Commit message: Updated URDF.

File: urdf/rover5.urdf (robot description, URDF)
Before this commit: robot rover5, 2 links, 1 joints
Links:
- link base_link: geometry visual mesh filename=package://rover5/meshes/rover5.dae scale=0.001 0.001 0.001

Commit message: Added STL.

File: urdf/rover5.urdf (robot description, URDF)
Before this commit: robot rover5, 2 links, 1 joints
Links:
- link base_link: geometry visual mesh filename=package://rover5/meshes/rover5.stl scale=0.001 0.001 0.001
